Commit message: removed comments causing errors in xacro processing and updated axes directions of joints 2 to 4

File: urdf/sketch_bot.urdf (robot description, URDF)
Before this commit: robot sketch_bot, 7 links, 6 joints
Links:
- added link tip
Joints:
- added joint tool0-tip: type fixed, parent tool0, child tip, origin xyz=0 -0.075 0 rpy=0 0 0
- joint joint_2: axis 1 0 0 -> -1 0 0
- joint joint_3: axis 1 0 0 -> -1 0 0
- joint joint_4: axis 1 0 0 -> -1 0 0

File: urdf/sketch_bot_macro.xacro (robot description, xacro)
@@ -1,5 +1,4 @@
 <?xml version="1.0"?>
 <robot xmlns:xacro="http://wiki.ros.org/xacro">
-  <!-- <xacro:include filename="$(find sketch_bot_resources)/urdf/common_materials.xacro"/> -->
   <material name="dark_yellow">
     <color rgba="0.75 0.55 0.15 1.0"/>
@@ -17,5 +16,4 @@
   <xacro:property name="yaw_offset" value="${radians(0)}"/>
   <xacro:macro name="sketch_bot" params="prefix">
-    <!-- links: main serial chain -->
     <link name="${prefix}base_link">
       <visual>
@@ -93,5 +91,4 @@
       </collision>
     </link>
-    <!-- joints: main serial chain -->
     <joint name="${prefix}joint_1" type="revolute">
       <origin xyz="0 0 0" rpy="0 0 0"/>
@@ -105,5 +102,5 @@
       <parent link="${prefix}link_1"/>
       <child link="${prefix}link_2"/>
-      <axis xyz="1 0 0"/>
+      <axis xyz="-1 0 0"/>
       <limit lower="${radians(-180)}" upper="${radians(180)}" effort="0" velocity="${radians(120)}"/>
     </joint>
@@ -112,5 +109,5 @@
       <parent link="${prefix}link_2"/>
       <child link="${prefix}link_3"/>
-      <axis xyz="1 0 0"/>
+      <axis xyz="-1 0 0"/>
       <limit lower="${radians(-180)}" upper="${radians(180)}" effort="0" velocity="${radians(120)}"/>
     </joint>
@@ -119,8 +116,7 @@
       <parent link="${prefix}link_3"/>
       <child link="${prefix}link_4"/>
-      <axis xyz="1 0 0"/>
+      <axis xyz="-1 0 0"/>
       <limit lower="${radians(-180)}" upper="${radians(180)}" effort="0" velocity="${radians(120)}"/>
     </joint>
-    <!-- ROS-Industrial 'tool0' frame: all-zeros tool frame -->
     <link name="${prefix}tool0" />
     <joint name="${prefix}link_4-tool0" type="fixed">
